File: BalancedSurroundOut.kicad_pcb (KiCad board)
At the start: 2 copper layers, 48 x 73 mm, 63 parts, among them IC1 TPS61252DSGT, IC2 DRV135UA_2K5, IC3 DRV135UA_2K5, J1 Conn_02x10_Odd_Even, J2 Conn_01x02, J3 XLR3_Ground, J4 XLR3_Ground, J5 Conn_01x03, J6 Conn_01x02, J8 Conn_01x03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

Commit message: refactor
Parts:
- removed J2: Conn_01x02, Connector_PinHeader_2.54mm:PinHeader_1x02_P2.54mm_Vertical
- added H1: MountingHole, MountingHole:MountingHole_3.2mm_M3, F.Cu at (148.0, 85.0)
- added H2: MountingHole, MountingHole:MountingHole_3.2mm_M3, F.Cu at (187.0, 85.0)
- added H3: MountingHole, MountingHole:MountingHole_3.2mm_M3, F.Cu at (187.0, 122.0)
- added H4: MountingHole, MountingHole:MountingHole_3.2mm_M3, F.Cu at (148.0, 122.0)
- J1: value Conn_02x10_Odd_Even -> Conn_02x06_Odd_Even; footprint Connector_PinHeader_2.54mm:PinHeader_2x10_P2.54mm_Vertical -> Connector_PinHeader_2.54mm:PinHeader_2x06_P2.54mm_Vertical
- moved J1 13.2 mm to (167.0, 122.0)
- moved C27 6.42 mm to (153.7, 113.2), turned to 90 degrees
- moved C24 4.13 mm to (172.2, 92.6)
- moved C23 4.04 mm to (171.5, 89.6)
- moved R10 4.03 mm to (168.2, 98.0)
- moved C10 4.03 mm to (182.0, 92.5)
- moved C11 4.03 mm to (173.5, 101.0)
- moved C12 4.03 mm to (173.0, 99.0)
- moved C13 4.03 mm to (173.2, 110.5)
- moved C14 4.03 mm to (162.5, 97.8)
- moved C15 4.03 mm to (177.7, 97.0)
- moved C16 4.03 mm to (175.2, 110.5)
- moved C17 4.03 mm to (169.2, 101.5)
- moved C18 4.03 mm to (176.0, 102.5)
- moved C19 4.03 mm to (168.5, 99.8)
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- renumbered JP3 to locked
Connections:
- J1 pad 1: /F3 -> VIN
- J1 pad 10: /MCLK -> /BCLK
- J1 pad 11: GND -> +3V3
- J1 pad 12: /LRCLK -> /DIN
- J1 pad 3: /F2 -> VIN
- J1 pad 4: +3V3 -> /DOUT
- J1 pad 5: /F1 -> unconnected-(J1-Pad5)
- J1 pad 6: GND -> /MCLK
- J1 pad 7: /F0 -> GND
- J1 pad 8: /DSDOE -> /LRCLK
- J1 pad 9: /D64 -> GND
Routing:
- net VIN: track 26.8 -> 1.14 mm
- net Net-(JP4-Pad2): track 28.3 -> 11.2 mm
- net +3V3: track 18.6 -> 25.5 mm
- net /BCLK: track 10.2 -> 15.8 mm
- net /DIN: track 11.3 -> 16.6 mm
- net GND: track 48.0 -> 43.6 mm, vias 73 -> 66
- net Net-(J4-Pad2): track 18.5 -> 14.4 mm
- net Net-(J4-Pad3): track 12.1 -> 8.11 mm
- net /DAC/LEFT: track 15.8 -> 12.0 mm
- net /DAC/RIGHT: track 13.3 -> 16.3 mm
- net /PowerSupply/SWITCH: track 0.00 -> 2.51 mm
- net /MCLK: track 4.45 -> 6.83 mm
- net Net-(J3-Pad3): track 3.46 -> 5.46 mm
- net Net-(J3-Pad2): track 8.52 -> 7.31 mm
- net /DAC/MCLK: track 5.95 -> 5.06 mm
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- added copper zone on B.Cu, net GND
- removed copper zone on F.Cu, net /PowerSupply/SWITCH
Other:
- board size 48 x 73 mm -> 45 x 62 mm
- board text removed: "GND"
- board text removed: "Vin"
- board text removed: "min 4.0V"

Commit message: latest
Parts:
- IC2, IC3: value DRV135UA_2K5 -> DRV134UA; footprint Package_SO:SOIC-8_3.9x4.9mm_P1.27mm -> BalancedAudioBox:SOIC127P1030X265-16N
- R3, R4: value 499k -> 510k
- moved R16 3.18 mm to (160.0, 83.5), turned to 0 degrees
- moved IC3 2.97 mm to (162.0, 89.8)
- moved JP4 2.91 mm to (164.2, 110.4), turned to 0 degrees
- moved J5 2.83 mm to (154.5, 89.7)
- moved R6 2.73 mm to (179.8, 83.5), turned to 180 degrees
- moved R10 2.50 mm to (165.8, 98.5), turned to 90 degrees
- moved R17 2.48 mm to (164.0, 83.5)
- moved R5 2.47 mm to (173.0, 83.5), turned to 180 degrees
- moved C10 2.30 mm to (184.2, 92.2)
- moved C9 2.28 mm to (184.2, 90.0)
- moved R9 2.28 mm to (174.8, 97.0)
- moved C7 1.80 mm to (185.8, 89.8)
- moved C8 1.78 mm to (185.8, 93.0)
- moved C24 1.63 mm to (170.6, 92.5)
- moved R1 1.57 mm to (151.4, 92.2)
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Connections:
- IC2 pad 1: /OutputDriver/LEFT_VON -> unconnected-(IC2-Pad1)
- IC2 pad 2: /OutputDriver/LEFT_VON -> unconnected-(IC2-Pad2)
- IC2 pad 3: GND -> /OutputDriver/LEFT_VON
- IC2 pad 4: /DAC/LEFT -> /OutputDriver/LEFT_VON
- IC2 pad 5: -5V -> GND
- IC2 pad 6: +5V -> /DAC/LEFT
- IC2 pad 7: /OutputDriver/LEFT_VOP -> unconnected-(IC2-Pad7)
- IC2 pad 8: /OutputDriver/LEFT_VOP -> unconnected-(IC2-Pad8)
- IC3 pad 1: /OutputDriver/RIGHT_VON -> unconnected-(IC3-Pad1)
- IC3 pad 2: /OutputDriver/RIGHT_VON -> unconnected-(IC3-Pad2)
- IC3 pad 3: GND -> /OutputDriver/RIGHT_VON
- IC3 pad 4: /DAC/RIGHT -> /OutputDriver/RIGHT_VON
- IC3 pad 5: -5V -> GND
- IC3 pad 6: +5V -> /DAC/RIGHT
- IC3 pad 7: /OutputDriver/RIGHT_VOP -> unconnected-(IC3-Pad7)
- IC3 pad 8: /OutputDriver/RIGHT_VOP -> unconnected-(IC3-Pad8)
- J3 pad 3: Net-(J3-Pad3) -> Net-(R5-Pad1)
- R16 pad 1: /OutputDriver/RIGHT_VON -> Net-(J4-Pad3)
- R16 pad 2: Net-(J4-Pad3) -> /OutputDriver/RIGHT_VON
- R5 pad 1: /OutputDriver/LEFT_VON -> Net-(R5-Pad1)
- R5 pad 2: Net-(J3-Pad3) -> /OutputDriver/LEFT_VON
Routing:
- net Net-(JP4-Pad2): track 11.2 -> 22.4 mm
- net +5V: track 53.7 -> 46.3 mm
- net Net-(R5-Pad1): track 0.00 -> 6.35 mm
- net GND: track 43.6 -> 49.6 mm
- net Net-(J3-Pad3): track 5.46 -> 0.00 mm
- net /OutputDriver/RIGHT_VON: track 3.09 -> 7.75 mm
- net /OutputDriver/LEFT_VON: track 3.59 -> 7.66 mm
- net Net-(J4-Pad3): track 8.11 -> 4.35 mm
- net /OutputDriver/RIGHT_VOP: track 4.36 -> 7.39 mm
- net Net-(R10-Pad2): track 6.22 -> 9.20 mm
- net Net-(J3-Pad2): track 7.31 -> 10.2 mm
- net /OutputDriver/LEFT_VOP: track 5.06 -> 7.75 mm
- net VIN: track 1.14 -> 3.70 mm
- net Net-(J4-Pad2): track 14.4 -> 16.7 mm
- net Net-(R9-Pad2): track 6.52 -> 8.79 mm
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
Commit message: ready for JLCPCB
Parts:
- added C29: 100n, Capacitor_SMD:C_0402_1005Metric, F.Cu at (178.7, 110.9)
- added U4: TLV75533PDBV, Package_TO_SOT_SMD:SOT-23-5, F.Cu at (177.5, 114.3)
- moved C1 0.35 mm to (156.0, 117.6)
- moved C24 0.20 mm to (170.6, 92.7)
- moved C27 0.20 mm to (153.5, 113.2)
Connections:
- net Net-(JP4-Pad2) renamed /DAC/5V
- J1 pad 10: /BCLK -> /DAC/DIN
- J1 pad 12: /DIN -> /DAC/LRCLK
- J1 pad 2: unconnected-(J1-Pad2) -> GND
- J1 pad 5: unconnected-(J1-Pad5) -> GND
- J1 pad 8: /LRCLK -> /DAC/BCLK
- U2 pad 13: /BCLK -> /DAC/BCLK
- U2 pad 14: /DIN -> /DAC/DIN
- U2 pad 15: /LRCLK -> /DAC/LRCLK
Routing:
- net /DAC/LRCLK: track 0.00 -> 16.8 mm
- net /DIN: track 16.6 -> 0.00 mm
- net /BCLK: track 15.8 -> 0.00 mm
- net /DAC/BCLK: track 0.00 -> 13.7 mm
- net /DAC/DIN: track 0.00 -> 13.7 mm
- net /LRCLK: track 12.6 -> 0.00 mm, vias 1 -> 0
- net /DAC/5V: track 22.4 -> 29.0 mm
- net GND: track 49.6 -> 53.8 mm, vias 66 -> 69
- net VIN: track 3.70 -> 4.49 mm
- net +3V3: track 25.5 -> 26.1 mm
- net +3.3VA: track 23.2 -> 22.7 mm
