File: BalancedSurroundOut.kicad_sch (KiCad schematic)
At the start: 4 parts, among them J1 Conn_02x10_Odd_Even, J2 Conn_01x02, J5 Conn_01x03

Commit message: refactor
Parts:
- removed J1: Conn_02x10_Odd_Even, Connector_PinHeader_2.54mm:PinHeader_2x10_P2.54mm_Vertical, symbol Connector_Generic:Conn_02x10_Odd_Even
- removed J2: Conn_01x02, Connector_PinHeader_2.54mm:PinHeader_1x02_P2.54mm_Vertical, symbol Connector_Generic:Conn_01x02
- added H1, H2, H3, H4: MountingHole, MountingHole:MountingHole_3.2mm_M3, symbol Mechanical:MountingHole
- added J1: Conn_02x06_Odd_Even, Connector_PinHeader_2.54mm:PinHeader_2x06_P2.54mm_Vertical, symbol Connector_Generic:Conn_02x06_Odd_Even
Connections:
- net +3V3: now also J1.2 (Pin_2)
- net BCLK: now also J1.10 (Pin_10)
- net DIN: now also J1.12 (Pin_12)
- net GND: now also J1.11 (Pin_11), J1.7 (Pin_7), J1.9 (Pin_9)
- net LRCLK: now also J1.8 (Pin_8)
- net MCLK: now also J1.6 (Pin_6)
- net VIN: now also J1.1 (Pin_1), J1.3 (Pin_3)
- new net DOUT: J1.4 (Pin_4)
- no-connect marks 8 -> 1

Commit message: latest
Connections:
- net +3V3: now also J1.11 (Pin_11); no longer J1.2 (Pin_2)
- net GND: no longer J1.11 (Pin_11)
Changed lines of the file:
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@@
 (kicad_sch (version 20211123) (generator eeschema)
   (paper "A4")
-  (junction (at 52.07 68.58) (diameter 0) (color 0 0 0 0)
-  )
   (junction (at 56.642 55.88) (diameter 0) (color 0 0 0 0)
   )
@@
     (stroke (width 0) (type default) (color 0 0 0 0))
   )
-  (wire (pts (xy 52.07 80.01) (xy 52.07 68.58))
-    (stroke (width 0) (type default) (color 0 0 0 0))
-  )
   (wire (pts (xy 74.93 58.42) (xy 87.63 58.42))
     (stroke (width 0) (type default) (color 0 0 0 0))
   )
-  (wire (pts (xy 52.07 68.58) (xy 62.23 68.58))
-    (stroke (width 0) (type default) (color 0 0 0 0))
-  )
   (wire (pts (xy 52.07 63.5) (xy 52.07 66.04))
     (stroke (width 0) (type default) (color 0 0 0 0))
@@
     (stroke (width 0) (type default) (color 0 0 0 0))
   )
+  (wire (pts (xy 62.23 68.58) (xy 42.926 68.58))
+    (stroke (width 0) (type default) (color 0 0 0 0))
+  )
   (wire (pts (xy 56.642 55.88) (xy 62.23 55.88))
     (stroke (width 0) (type default) (color 0 0 0 0))
@@
     (stroke (width 0) (type default) (color 0 0 0 0))
   )
-  (wire (pts (xy 81.28 55.88) (xy 81.28 46.99))
-    (stroke (width 0) (type default) (color 0 0 0 0))
-  )
   (wire (pts (xy 207.01 143.51) (xy 224.79 143.51))
     (stroke (width 0) (type default) (color 0 0 0 0))
@@
     (stroke (width 0) (type default) (color 0 0 0 0))
   )
+  (wire (pts (xy 42.926 68.58) (xy 42.926 46.482))
+    (stroke (width 0) (type default) (color 0 0 0 0))
+  )
   (wire (pts (xy 62.23 66.04) (xy 52.07 66.04))
     (stroke (width 0) (type default) (color 0 0 0 0))
@@
     (stroke (width 0) (type default) (color 0 0 0 0))
   )
-  (wire (pts (xy 74.93 55.88) (xy 81.28 55.88))
-    (stroke (width 0) (type default) (color 0 0 0 0))
-  )
   (wire (pts (xy 224.79 143.51) (xy 224.79 133.35))
     (stroke (width 0) (type default) (color 0 0 0 0))
@@
     (stroke (width 0) (type default) (color 0 0 0 0))
   )
-  (wire (pts (xy 52.07 66.04) (xy 52.07 68.58))
+  (wire (pts (xy 52.07 66.04) (xy 52.07 80.01))
     (stroke (width 0) (type default) (color 0 0 0 0))
   )
@@
     (pin "1")
   )
-  (symbol (lib_id "power:+3.3V") (at 81.28 46.99 0) (unit 1)
+  (symbol (lib_id "power:+3.3V") (at 42.926 46.482 0) (unit 1)
     (in_bom yes) (on_board yes)
-    (property "Reference" "#PWR02" (id 0) (at 81.28 50.8 0)
-      (effects (font (size 1.27 1.27)) hide)
-    )
-    (property "Value" "+3.3V" (id 1) (at 81.661 42.5958 0))
-    (property "Footprint" "" (id 2) (at 81.28 46.99 0)
-      (effects (font (size 1.27 1.27)) hide)
-    )
-    (property "Datasheet" "" (id 3) (at 81.28 46.99 0)
+    (property "Reference" "#PWR02" (id 0) (at 42.926 50.292 0)
+      (effects (font (size 1.27 1.27)) hide)
+    )
+    (property "Value" "+3.3V" (id 1) (at 43.307 42.0878 0))
+    (property "Footprint" "" (id 2) (at 42.926 46.482 0)
+      (effects (font (size 1.27 1.27)) hide)
+    )
+    (property "Datasheet" "" (id 3) (at 42.926 46.482 0)
       (effects (font (size 1.27 1.27)) hide)
     )
@@
       (reference "IC1") (unit 1) (value "TPS61252DSGT") (footprint "BalancedAudioBox:SON50P200X200X80-9N")
     )
-    (path "/00000000-0000-0000-0000-00005d3d9e6f/00000000-0000-0000-0000-00005d3da719"
-      (reference "IC2") (unit 1) (value "DRV135UA_2K5") (footprint "Package_SO:SOIC-8_3.9x4.9mm_P1.27mm")
-    )
-    (path "/00000000-0000-0000-0000-00005d3d9e6f/00000000-0000-0000-0000-00005d40e195"
-      (reference "IC3") (unit 1) (value "DRV135UA_2K5") (footprint "Package_SO:SOIC-8_3.9x4.9mm_P1.27mm")
+    (path "/00000000-0000-0000-0000-00005d3d9e6f/f9e7a6a4-92a5-486e-8c4b-6e5000231ed6"
+      (reference "IC2") (unit 1) (value "DRV134UA") (footprint "SOIC127P1030X265-16N")
+    )
+    (path "/00000000-0000-0000-0000-00005d3d9e6f/8212be8e-110b-4617-984e-20e0f6bc0c8a"
+      (reference "IC3") (unit 1) (value "DRV134UA") (footprint "SOIC127P1030X265-16N")
     )
     (path "/677544df-385f-472d-9798-c5c06019f8c0"
@@
     )
     (path "/00000000-0000-0000-0000-00005d3d9e16/00000000-0000-0000-0000-00005d3fb5b1"
-      (reference "R3") (unit 1) (value "499k") (footprint "Resistor_SMD:R_0402_1005Metric")
+      (reference "R3") (unit 1) (value "510k") (footprint "Resistor_SMD:R_0402_1005Metric")
     )
     (path "/00000000-0000-0000-0000-00005d3d9e16/00000000-0000-0000-0000-00005d3f8f3f"
-      (reference "R4") (unit 1) (value "499k") (footprint "Resistor_SMD:R_0402_1005Metric")
+      (reference "R4") (unit 1) (value "510k") (footprint "Resistor_SMD:R_0402_1005Metric")
     )
     (path "/00000000-0000-0000-0000-00005d3d9e6f/00000000-0000-0000-0000-00005d3dd7c6"

Commit message: ready for JLCPCB
Parts:
- J5: now left out of the parts list
Connections:
- net GND: now also J1.2 (Pin_2), J1.5 (Pin_5)
- net BCLK renamed DAC/DIN
- net DIN renamed DAC/LRCLK
- net LRCLK renamed DAC/BCLK
- no-connect marks 1 -> 0
Changed lines of the file:
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@@
 (kicad_sch (version 20211123) (generator eeschema)
   (paper "A4")
+  (junction (at 52.07 63.5) (diameter 0) (color 0 0 0 0)
+  )
   (junction (at 56.642 55.88) (diameter 0) (color 0 0 0 0)
   )
   (junction (at 52.07 66.04) (diameter 0) (color 0 0 0 0)
   )
-  (no_connect (at 87.63 58.42))
-  (wire (pts (xy 74.93 63.5) (xy 105.41 63.5))
-    (stroke (width 0) (type default) (color 0 0 0 0))
-  )
-  (wire (pts (xy 74.93 68.58) (xy 105.41 68.58))
-    (stroke (width 0) (type default) (color 0 0 0 0))
+  (junction (at 52.07 75.184) (diameter 0) (color 0 0 0 0)
   )
   (wire (pts (xy 160.02 54.61) (xy 189.23 54.61))
@@
     (stroke (width 0) (type default) (color 0 0 0 0))
   )
-  (wire (pts (xy 74.93 58.42) (xy 87.63 58.42))
+  (wire (pts (xy 74.93 66.04) (xy 79.502 66.04))
+    (stroke (width 0) (type default) (color 0 0 0 0))
+  )
+  (wire (pts (xy 74.93 58.42) (xy 79.756 58.42))
+    (stroke (width 0) (type default) (color 0 0 0 0))
+  )
+  (wire (pts (xy 77.216 75.184) (xy 52.07 75.184))
+    (stroke (width 0) (type default) (color 0 0 0 0))
+  )
+  (wire (pts (xy 96.266 63.5) (xy 96.266 68.58))
+    (stroke (width 0) (type default) (color 0 0 0 0))
+  )
+  (wire (pts (xy 79.502 66.04) (xy 79.502 70.612))
     (stroke (width 0) (type default) (color 0 0 0 0))
   )
@@
     (stroke (width 0) (type default) (color 0 0 0 0))
   )
+  (wire (pts (xy 77.216 55.88) (xy 77.216 75.184))
+    (stroke (width 0) (type default) (color 0 0 0 0))
+  )
   (wire (pts (xy 207.01 138.43) (xy 215.9 138.43))
     (stroke (width 0) (type default) (color 0 0 0 0))
   )
+  (wire (pts (xy 91.186 66.04) (xy 91.186 63.5))
+    (stroke (width 0) (type default) (color 0 0 0 0))
+  )
   (wire (pts (xy 62.23 58.42) (xy 56.642 58.42))
     (stroke (width 0) (type default) (color 0 0 0 0))
   )
+  (wire (pts (xy 62.23 60.96) (xy 52.07 60.96))
+    (stroke (width 0) (type default) (color 0 0 0 0))
+  )
   (wire (pts (xy 207.01 143.51) (xy 224.79 143.51))
     (stroke (width 0) (type default) (color 0 0 0 0))
   )
+  (wire (pts (xy 99.822 68.58) (xy 99.822 70.612))
+    (stroke (width 0) (type default) (color 0 0 0 0))
+  )
+  (wire (pts (xy 91.186 63.5) (xy 74.93 63.5))
+    (stroke (width 0) (type default) (color 0 0 0 0))
+  )
   (wire (pts (xy 62.23 63.5) (xy 52.07 63.5))
     (stroke (width 0) (type default) (color 0 0 0 0))
   )
-  (wire (pts (xy 105.41 66.04) (xy 74.93 66.04))
+  (wire (pts (xy 52.07 60.96) (xy 52.07 63.5))
     (stroke (width 0) (type default) (color 0 0 0 0))
   )
@@
     (stroke (width 0) (type default) (color 0 0 0 0))
   )
+  (wire (pts (xy 105.41 63.5) (xy 96.266 63.5))
+    (stroke (width 0) (type default) (color 0 0 0 0))
+  )
+  (wire (pts (xy 52.07 75.184) (xy 52.07 80.01))
+    (stroke (width 0) (type default) (color 0 0 0 0))
+  )
   (wire (pts (xy 215.9 138.43) (xy 215.9 133.35))
     (stroke (width 0) (type default) (color 0 0 0 0))
   )
+  (wire (pts (xy 105.41 66.04) (xy 91.186 66.04))
+    (stroke (width 0) (type default) (color 0 0 0 0))
+  )
   (wire (pts (xy 215.9 140.97) (xy 215.9 153.67))
     (stroke (width 0) (type default) (color 0 0 0 0))
@@
     (stroke (width 0) (type default) (color 0 0 0 0))
   )
+  (wire (pts (xy 96.266 68.58) (xy 74.93 68.58))
+    (stroke (width 0) (type default) (color 0 0 0 0))
+  )
+  (wire (pts (xy 74.93 55.88) (xy 77.216 55.88))
+    (stroke (width 0) (type default) (color 0 0 0 0))
+  )
   (wire (pts (xy 224.79 143.51) (xy 224.79 133.35))
     (stroke (width 0) (type default) (color 0 0 0 0))
   )
+  (wire (pts (xy 99.822 68.58) (xy 105.41 68.58))
+    (stroke (width 0) (type default) (color 0 0 0 0))
+  )
   (wire (pts (xy 97.79 43.18) (xy 97.79 38.1))
     (stroke (width 0) (type default) (color 0 0 0 0))
   )
-  (wire (pts (xy 52.07 66.04) (xy 52.07 80.01))
+  (wire (pts (xy 52.07 66.04) (xy 52.07 75.184))
     (stroke (width 0) (type default) (color 0 0 0 0))
   )
   (wire (pts (xy 160.02 57.15) (xy 189.23 57.15))
+    (stroke (width 0) (type default) (color 0 0 0 0))
+  )
+  (wire (pts (xy 99.822 70.612) (xy 79.502 70.612))
     (stroke (width 0) (type default) (color 0 0 0 0))
   )
@@
     (effects (font (size 1.27 1.27)) (justify left bottom))
   )
-  (label "LRCLK" (at 86.36 63.5 0)
-    (effects (font (size 1.27 1.27)) (justify left bottom))
-  )
   (label "MCLK" (at 86.36 60.96 0)
     (effects (font (size 1.27 1.27)) (justify left bottom))
   )
-  (label "DIN" (at 86.36 68.58 0)
-    (effects (font (size 1.27 1.27)) (justify left bottom))
-  )
-  (label "BCLK" (at 86.36 66.04 0)
-    (effects (font (size 1.27 1.27)) (justify left bottom))
-  )
-  (label "DOUT" (at 87.63 58.42 0)
+  (label "DOUT" (at 79.756 58.42 0)
     (effects (font (size 1.27 1.27)) (justify left bottom))
   )
@@
   )
   (symbol (lib_id "Connector_Generic:Conn_01x03") (at 201.93 140.97 0) (mirror y) (unit 1)
-    (in_bom yes) (on_board yes)
+    (in_bom no) (on_board yes)
     (property "Reference" "J5" (id 0) (at 204.0128 132.9182 0))
     (property "Value" "Conn_01x03" (id 1) (at 204.0128 135.2296 0))
@@
       (reference "#PWR080") (unit 1) (value "+3.3VA") (footprint "")
     )
+    (path "/00000000-0000-0000-0000-00005d41da57/d3bb72e4-ca01-454b-a788-f17eadb0dcb1"
+      (reference "#PWR0101") (unit 1) (value "GND") (footprint "")
+    )
+    (path "/00000000-0000-0000-0000-00005d41da57/c656dddf-310f-41eb-ab3a-c91aaf30bd56"
+      (reference "#PWR0102") (unit 1) (value "+3.3V") (footprint "")
+    )
     (path "/00000000-0000-0000-0000-00005d3d9e6f/00000000-0000-0000-0000-00005d47842a"
       (reference "#PWR0103") (unit 1) (value "GND") (footprint "")
@@
       (reference "#PWR0104") (unit 1) (value "+3.3VA") (footprint "")
     )
+    (path "/00000000-0000-0000-0000-00005d41da57/01372e87-4188-4514-9591-edf8c5b99d69"
+      (reference "#PWR0105") (unit 1) (value "GND") (footprint "")
+    )
     (path "/00000000-0000-0000-0000-00005d3d9e16/00000000-0000-0000-0000-00005d41488c"
       (reference "C1") (unit 1) (value "10u/25V") (footprint "Capacitor_SMD:C_0805_2012Metric")
@@
       (reference "C28") (unit 1) (value "100n") (footprint "Capacitor_SMD:C_0402_1005Metric")
     )
+    (path "/00000000-0000-0000-0000-00005d41da57/ed878fee-8763-4db2-9e0d-021b5307da37"
+      (reference "C29") (unit 1) (value "100n") (footprint "Capacitor_SMD:C_0402_1005Metric")
+    )
     (path "/d14e12ba-93b8-4d62-988f-5b00b14ea0d1"
       (reference "H1") (unit 1) (value "MountingHole") (footprint "MountingHole:MountingHole_3.2mm_M3")
@@
       (reference "U3") (unit 1) (value "TLV75533PDBV") (footprint "Package_TO_SOT_SMD:SOT-23-5")
     )
-  )
+    (path "/00000000-0000-0000-0000-00005d41da57/6f3671a4-0be9-4e1e-8c4f-fbff29ecc76e"
+      (reference "U4") (unit 1) (value "TLV75533PDBV") (footprint "Package_TO_SOT_SMD:SOT-23-5")
+    )
+  )
