File: DAC.kicad_sch (KiCad schematic)
At the start: 21 parts, among them U2 PCM5102, U3 TLV75533PDBV

Commit message: ready for JLCPCB
Parts:
- added C29: 100n, Capacitor_SMD:C_0402_1005Metric, symbol Device:C
- added U4: TLV75533PDBV, Package_TO_SOT_SMD:SOT-23-5, symbol Regulator_Linear:TLV75533PDBV
- C11, C12: LCSC (none) -> C49217
- C16, C17, C18, C28: LCSC (none) -> C307331
Connections:
- net +3V3: now also C29.1, U4.5 (OUT)
- net GND: now also C29.2, U4.2 (GND)
- net 5V: now reaches JP4.2 (C), R7.1, U3.1 (IN), U3.3 (EN)
- net 5V: now also U4.1 (IN), U4.3 (EN)
Changed lines of the file:
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@@
   (junction (at 194.31 78.74) (diameter 0) (color 0 0 0 0)
   )
+  (junction (at 230.378 32.766) (diameter 0) (color 0 0 0 0)
+  )
   (junction (at 138.43 114.3) (diameter 0) (color 0 0 0 0)
   )
@@
   (junction (at 184.15 86.36) (diameter 0) (color 0 0 0 0)
   )
+  (junction (at 212.09 32.766) (diameter 0) (color 0 0 0 0)
+  )
   (junction (at 81.28 101.6) (diameter 0) (color 0 0 0 0)
   )
@@
     (stroke (width 0) (type default) (color 0 0 0 0))
   )
+  (wire (pts (xy 212.09 32.766) (xy 212.09 35.306))
+    (stroke (width 0) (type default) (color 0 0 0 0))
+  )
   (wire (pts (xy 135.89 111.76) (xy 135.89 114.3))
     (stroke (width 0) (type default) (color 0 0 0 0))
@@
     (stroke (width 0) (type default) (color 0 0 0 0))
   )
+  (wire (pts (xy 227.33 32.766) (xy 230.378 32.766))
+    (stroke (width 0) (type default) (color 0 0 0 0))
+  )
   (wire (pts (xy 101.6 66.04) (xy 101.6 62.23))
     (stroke (width 0) (type default) (color 0 0 0 0))
   )
+  (wire (pts (xy 230.378 44.196) (xy 230.378 40.386))
+    (stroke (width 0) (type default) (color 0 0 0 0))
+  )
   (wire (pts (xy 120.65 118.11) (xy 120.65 104.14))
     (stroke (width 0) (type default) (color 0 0 0 0))
@@
     (stroke (width 0) (type default) (color 0 0 0 0))
   )
+  (wire (pts (xy 204.47 32.766) (xy 212.09 32.766))
+    (stroke (width 0) (type default) (color 0 0 0 0))
+  )
   (wire (pts (xy 151.13 99.06) (xy 157.48 99.06))
     (stroke (width 0) (type default) (color 0 0 0 0))
@@
   (label "DEEMP" (at 110.49 110.49 0)
     (effects (font (size 1.27 1.27)) (justify left bottom))
+  )
+  (label "5V" (at 204.47 32.766 0)
+    (effects (font (size 1.27 1.27)) (justify left bottom))
+  )
+  (label "5V" (at 81.28 54.61 180)
+    (effects (font (size 1.27 1.27)) (justify right bottom))
   )
   (global_label "+5.4V" (shape input) (at 76.2 63.5 270) (fields_autoplaced)
@@
       (effects (font (size 1.27 1.27)) hide)
     )
+    (property "LCSC" "C49217" (id 4) (at 157.48 95.25 0)
+      (effects (font (size 1.27 1.27)) hide)
+    )
     (pin "1")
     (pin "2")
@@
     )
     (property "Datasheet" "~" (id 3) (at 157.48 113.03 0)
+      (effects (font (size 1.27 1.27)) hide)
+    )
+    (property "LCSC" "C49217" (id 4) (at 157.48 113.03 0)
       (effects (font (size 1.27 1.27)) hide)
     )
@@
       (effects (font (size 1.27 1.27)) hide)
     )
+    (property "LCSC" "C307331" (id 4) (at 226.06 109.22 0)
+      (effects (font (size 1.27 1.27)) hide)
+    )
     (pin "1")
     (pin "2")
@@
       (effects (font (size 1.27 1.27)) hide)
     )
+    (property "LCSC" "C307331" (id 4) (at 247.65 109.22 0)
+      (effects (font (size 1.27 1.27)) hide)
+    )
     (pin "1")
     (pin "2")
@@
     )
     (property "Datasheet" "~" (id 3) (at 226.06 142.24 0)
+      (effects (font (size 1.27 1.27)) hide)
+    )
+    (property "LCSC" "C307331" (id 4) (at 226.06 142.24 0)
       (effects (font (size 1.27 1.27)) hide)
     )
@@
     )
     (property "Datasheet" "~" (id 3) (at 101.6 58.42 0)
+      (effects (font (size 1.27 1.27)) hide)
+    )
+    (property "LCSC" "C307331" (id 4) (at 101.6 58.42 0)
       (effects (font (size 1.27 1.27)) hide)
     )
@@
     (pin "5")
   )
+  (symbol (lib_id "power:GND") (at 219.71 42.926 0) (unit 1)
+    (in_bom yes) (on_board yes)
+    (property "Reference" "#PWR0105" (id 0) (at 219.71 49.276 0)
+      (effects (font (size 1.27 1.27)) hide)
+    )
+    (property "Value" "GND" (id 1) (at 219.837 47.3202 0))
+    (property "Footprint" "" (id 2) (at 219.71 42.926 0)
+      (effects (font (size 1.27 1.27)) hide)
+    )
+    (property "Datasheet" "" (id 3) (at 219.71 42.926 0)
+      (effects (font (size 1.27 1.27)) hide)
+    )
+    (pin "1")
+  )
+  (symbol (lib_id "Regulator_Linear:TLV75533PDBV") (at 219.71 35.306 0) (unit 1)
+    (in_bom yes) (on_board yes)
+    (property "Reference" "U4" (id 0) (at 219.71 26.6192 0))
+    (property "Value" "TLV75533PDBV" (id 1) (at 219.71 28.9306 0))
+    (property "Footprint" "Package_TO_SOT_SMD:SOT-23-5" (id 2) (at 219.71 27.686 0)
+      (effects (font (size 1.27 1.27) italic) hide)
+    )
+    (property "Datasheet" "http://www.ti.com/lit/ds/symlink/tlv755p.pdf" (id 3) (at 219.71 35.306 0)
+      (effects (font (size 1.27 1.27)) hide)
+    )
+    (pin "1")
+    (pin "2")
+    (pin "3")
+    (pin "4")
+    (pin "5")
+  )
+  (symbol (lib_id "power:+3.3V") (at 230.378 32.766 0) (unit 1)
+    (in_bom yes) (on_board yes)
+    (property "Reference" "#PWR0102" (id 0) (at 230.378 36.576 0)
+      (effects (font (size 1.27 1.27)) hide)
+    )
+    (property "Value" "+3.3V" (id 1) (at 230.759 28.3718 0))
+    (property "Footprint" "" (id 2) (at 230.378 32.766 0)
+      (effects (font (size 1.27 1.27)) hide)
+    )
+    (property "Datasheet" "" (id 3) (at 230.378 32.766 0)
+      (effects (font (size 1.27 1.27)) hide)
+    )
+    (pin "1")
+  )
+  (symbol (lib_id "power:GND") (at 230.378 44.196 0) (unit 1)
+    (in_bom yes) (on_board yes)
+    (property "Reference" "#PWR0101" (id 0) (at 230.378 50.546 0)
+      (effects (font (size 1.27 1.27)) hide)
+    )
+    (property "Value" "GND" (id 1) (at 230.505 48.5902 0))
+    (property "Footprint" "" (id 2) (at 230.378 44.196 0)
+      (effects (font (size 1.27 1.27)) hide)
+    )
+    (property "Datasheet" "" (id 3) (at 230.378 44.196 0)
+      (effects (font (size 1.27 1.27)) hide)
+    )
+    (pin "1")
+  )
+  (symbol (lib_id "Device:C") (at 230.378 36.576 0) (unit 1)
+    (in_bom yes) (on_board yes)
+    (property "Reference" "C29" (id 0) (at 233.299 35.4076 0)
+      (effects (font (size 1.27 1.27)) (justify left))
+    )
+    (property "Value" "100n" (id 1) (at 233.299 37.719 0)
+      (effects (font (size 1.27 1.27)) (justify left))
+    )
+    (property "Footprint" "Capacitor_SMD:C_0402_1005Metric" (id 2) (at 231.3432 40.386 0)
+      (effects (font (size 1.27 1.27)) hide)
+    )
+    (property "Datasheet" "~" (id 3) (at 230.378 36.576 0)
+      (effects (font (size 1.27 1.27)) hide)
+    )
+    (property "LCSC" "C307331" (id 4) (at 230.378 36.576 0)
+      (effects (font (size 1.27 1.27)) hide)
+    )
+    (pin "1")
+    (pin "2")
+  )
 )
