File: OutputDriver.kicad_sch (KiCad schematic)
At the start: 17 parts, among them IC2 DRV135UA_2K5, IC3 DRV135UA_2K5, J3 XLR3_Ground, J4 XLR3_Ground, J8 Conn_01x03

Commit message: latest
Parts:
- removed IC2, IC3: DRV135UA_2K5, Package_SO:SOIC-8_3.9x4.9mm_P1.27mm, symbol BalancedAudioBox:DRV135UA_2K5
- added IC2, IC3: DRV134UA, SOIC127P1030X265-16N, symbol BalancedAudioBox:DRV134UA
Connections:
- net +5V: now also IC2.12 (V+), IC3.12 (V+)
- net -5V: now also IC2.11 (V-), IC3.11 (V-)
- net GND: now also IC2.5 (GND), IC3.5 (GND)
- net LEFT: now also IC2.6 (VIN)
- net LEFT_VON: now also R5.2, IC2.3 (-V_O), IC2.4 (-SENSE); no longer R5.1
- net LEFT_VOP: now also IC2.13 (+SENSE), IC2.14 (+VO)
- net RIGHT: now also IC3.6 (VIN)
- net RIGHT_VON: now also R16.2, IC3.3 (-V_O), IC3.4 (-SENSE); no longer R16.1
- net RIGHT_VOP: now also IC3.13 (+SENSE), IC3.14 (+VO)
- net at J3.3: now also R5.1; no longer R5.2
- net at J4.3: now also R16.1; no longer R16.2
- no-connect marks 0 -> 16
Other:
- moved on the sheet: R16, R5

Commit message: ready for JLCPCB
Parts:
- J3, J4, J8: now left out of the parts list
Changed lines of the file:
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@@
   )
   (symbol (lib_id "Connector:XLR3_Ground") (at 80.01 41.91 0) (unit 1)
-    (in_bom yes) (on_board yes)
+    (in_bom no) (on_board yes)
     (property "Reference" "J3" (id 0) (at 80.01 32.639 0))
     (property "Value" "XLR3_Ground" (id 1) (at 80.01 34.9504 0))
@@
   )
   (symbol (lib_id "Connector:XLR3_Ground") (at 80.01 116.84 0) (unit 1)
-    (in_bom yes) (on_board yes)
+    (in_bom no) (on_board yes)
     (property "Reference" "J4" (id 0) (at 80.01 107.569 0))
     (property "Value" "XLR3_Ground" (id 1) (at 80.01 109.8804 0))
@@
   )
   (symbol (lib_id "Connector_Generic:Conn_01x03") (at 49.53 109.22 0) (mirror y) (unit 1)
-    (in_bom yes) (on_board yes)
+    (in_bom no) (on_board yes)
     (property "Reference" "J8" (id 0) (at 51.6128 101.1682 0))
     (property "Value" "Conn_01x03" (id 1) (at 51.6128 103.4796 0))
