File: PowerSupply.kicad_sch (KiCad schematic)
At the start: 21 parts, among them IC1 TPS61252DSGT, J6 Conn_01x02, U1 LM27762

Commit message: latest
Parts:
- IC1: LCSC (none) -> C128617
- R1, R2: LCSC (none) -> C477217
- R14: LCSC (none) -> C228942
- R15: LCSC (none) -> C25760
- R3, R4: value 499k -> 510k; LCSC (none) -> C11616
Other:
- note added: "target: 499k, rounded to basic part"
Changed lines of the file:
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@@
+    (effects (font (size 1.27 1.27)) (justify left bottom))
+  )
+  (text "target: 499k, rounded to basic part" (at 279.146 123.19 90)
     (effects (font (size 1.27 1.27)) (justify left bottom))
   )
@@
     (property "RS Price/Stock" "http://uk.rs-online.com/web/p/products/7300675P" (id 11) (at 67.31 104.14 0)
       (effects (font (size 1.27 1.27)) (justify left) hide)
+    )
+    (property "LCSC" "C128617" (id 12) (at 93.98 83.82 0)
+      (effects (font (size 1.27 1.27)) hide)
     )
     (pin "1")
@@
       (effects (font (size 1.27 1.27)) hide)
     )
+    (property "LCSC" "C228942" (id 4) (at 118.11 91.44 0)
+      (effects (font (size 1.27 1.27)) hide)
+    )
     (pin "1")
     (pin "2")
@@
     )
     (property "Datasheet" "~" (id 3) (at 118.11 104.14 0)
+      (effects (font (size 1.27 1.27)) hide)
+    )
+    (property "LCSC" "C25760" (id 4) (at 118.11 104.14 0)
       (effects (font (size 1.27 1.27)) hide)
     )
@@
       (effects (font (size 1.27 1.27)) hide)
     )
+    (property "LCSC" "C477217" (id 4) (at 267.97 106.68 0)
+      (effects (font (size 1.27 1.27)) hide)
+    )
     (pin "1")
     (pin "2")
@@
       (effects (font (size 1.27 1.27)) (justify left))
     )
-    (property "Value" "499k" (id 1) (at 269.748 116.713 0)
+    (property "Value" "510k" (id 1) (at 269.748 116.713 0)
       (effects (font (size 1.27 1.27)) (justify left))
     )
@@
       (effects (font (size 1.27 1.27)) hide)
     )
+    (property "LCSC" "C11616" (id 4) (at 267.97 115.57 0)
+      (effects (font (size 1.27 1.27)) hide)
+    )
     (pin "1")
     (pin "2")
@@
       (effects (font (size 1.27 1.27)) hide)
     )
+    (property "LCSC" "C477217" (id 4) (at 250.19 106.68 0)
+      (effects (font (size 1.27 1.27)) hide)
+    )
     (pin "1")
     (pin "2")
@@
       (effects (font (size 1.27 1.27)) (justify left))
     )
-    (property "Value" "499k" (id 1) (at 251.968 116.713 0)
+    (property "Value" "510k" (id 1) (at 251.968 116.713 0)
       (effects (font (size 1.27 1.27)) (justify left))
     )
@@
       (effects (font (size 1.27 1.27)) hide)
     )
+    (property "LCSC" "C11616" (id 4) (at 250.19 115.57 0)
+      (effects (font (size 1.27 1.27)) hide)
+    )

Commit message: ready for JLCPCB
Parts:
- J6: now left out of the parts list
Changed lines of the file:
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@@
     (effects (font (size 1.27 1.27)) (justify left bottom))
   )
-  (label "PGOOD" (at 165.1 91.44 0)
-    (effects (font (size 1.27 1.27)) (justify left bottom))
-  )
   (label "ILIM" (at 93.98 91.44 0)
-    (effects (font (size 1.27 1.27)) (justify left bottom))
-  )
-  (label "OUT-" (at 205.74 101.6 0)
     (effects (font (size 1.27 1.27)) (justify left bottom))
   )
@@
   )
   (symbol (lib_id "Connector_Generic:Conn_01x02") (at 139.7 77.47 0) (unit 1)
-    (in_bom yes) (on_board yes)
+    (in_bom no) (on_board yes)
     (property "Reference" "J6" (id 0) (at 141.732 77.6732 0)
       (effects (font (size 1.27 1.27)) (justify left))

Commit message: smth
Parts:
- R14: LCSC C228942 -> C27014
Changed lines of the file:
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@@
       (effects (font (size 1.27 1.27)) hide)
     )
-    (property "LCSC" "C228942" (id 4) (at 118.11 91.44 0)
+    (property "LCSC" "C27014" (id 4) (at 118.11 91.44 0)
       (effects (font (size 1.27 1.27)) hide)
     )
